File: pcb/kamaji.sch (KiCad schematic (older format))
At the start: 31 parts, among them J1 RJ10, J2 RJ10, J3 RJ10, J4 RJ10, Q1 IRF540N, SW1 CTRL1, SW2 CTRL2, SW3 CTRL3, U1 ATMEGA328P-PU, Y1 Crystal

Commit message: lay out the 1.1 PCB
Connections:
- net CBTN1: now also U1.23 ((PCINT8/ADC0)PC0); no longer U1.16 ((PCINT2/OC1B/~SS~)PB2)
- net LCD_RS: now also U1.16 ((PCINT2/OC1B/~SS~)PB2); no longer U1.23 ((PCINT8/ADC0)PC0)
- net PBTN1: now also U1.3 ((PCINT17/TXD)PD1); no longer U1.2 ((PCINT16/RXD)PD0)
- net PBTN2: now also U1.5 ((PCINT19/OC2B/INT1)PD3); no longer U1.4 ((PCINT18/INT0)PD2)
- net PLED1: now also U1.2 ((PCINT16/RXD)PD0); no longer U1.3 ((PCINT17/TXD)PD1)
- net PLED2: now also U1.4 ((PCINT18/INT0)PD2); no longer U1.5 ((PCINT19/OC2B/INT1)PD3)
Changed lines of the file:
@@
 Text GLabel 4325 3000 2    60   Input ~ 0
 RST
+Text GLabel 3675 3250 2    60   Input ~ 0
+PBTN1
 Text GLabel 3275 3150 2    60   Input ~ 0
-PBTN1
-Text GLabel 3675 3250 2    60   Input ~ 0
 PLED1
+Text GLabel 3675 3450 2    60   Input ~ 0
+PBTN2
 Text GLabel 3275 3350 2    60   Input ~ 0
-PBTN2
-Text GLabel 3675 3450 2    60   Input ~ 0
 PLED2
 Text GLabel 3275 3550 2    60   Input ~ 0
@@
 Text GLabel 4175 1700 2    60   Input ~ 0
 CBTN2
-Text GLabel 3250 1750 2    60   Input ~ 0
+Text GLabel 3275 2400 2    60   Input ~ 0
 CBTN1
 $Comp
@@
 Text GLabel 6725 3150 3    60   Input ~ 0
 LCD_D0
-Text GLabel 3275 2400 2    60   Input ~ 0
+Text GLabel 3250 1750 2    60   Input ~ 0
 LCD_RS
 Text GLabel 3675 2500 2    60   Input ~ 0
