File: pcb/1.0/kamaji.sch (KiCad schematic (older format))
At the start: 30 parts, among them J1 RJ10, J2 RJ10, J3 RJ10, J4 RJ10, J5 RJ10, Q1 IRF540N, SW1 CTRL1, SW2 CTRL2, SW3 CTRL3, U1 ATMEGA328P-PU

Commit message: update title on 1.0 schematic
Parts:
- DS1: symbol LCD-016N002L -> LCD-016N002L-RESCUE-kamaji
- Q1: symbol IRF540N -> IRF540N-RESCUE-kamaji
Changed lines of the file:
@@
 EESchema Schematic File Version 2
+LIBS:kamaji-rescue
 LIBS:power
 LIBS:device
@@
 LIBS:ftdi
 LIBS:gennum
-LIBS:graphic
 LIBS:hc11
 LIBS:intersil
@@
 LIBS:Lattice
 LIBS:leds
-LIBS:logo
 LIBS:maxim
 LIBS:mechanical
@@
 Date ""
 Rev "1.0"
-Comp "Dead Man's Bluff Inc."
+Comp ""
 Comment1 "© Ilya Strukov <iley@iley.ru>"
 Comment2 ""
@@
 $EndComp
 $Comp
-L LCD-016N002L DS1
+L LCD-016N002L-RESCUE-kamaji DS1
 U 1 1 596C4BC3
 P 6475 2050
@@
 $EndComp
 $Comp
-L IRF540N Q1
+L IRF540N-RESCUE-kamaji Q1
 U 1 1 5973C5BD
 P 9650 5450
