File: pcb/2.0/_saved_kamaji.sch (KiCad schematic (older format))
At the start: 53 parts, among them J1 RJ10, J2 RJ10, J3 RJ10, J4 RJ10, J5 RJ10, J6 RJ10, J7 USB_B, J8 USB_A, Q1 2N3904, Q2 IRL540N, Q3 IRL540N, SW1 SW_Push, SW2 SW_Push, SW3 SW_Push, U1 ATMEGA32U4-AU, Y1 16MHz

Commit message: change socket and potentiometer footprints
Parts:
- J8: footprint Connectors:USB_A -> kamaji:USB_A
Changed lines of the file:
@@
 F 0 "J8" H 10100 5060 50  0000 L CNN
 F 1 "USB_A" H 10100 4960 50  0000 L CNN
-F 2 "Connectors:USB_A" H 10450 4560 50  0001 C CNN
+F 2 "kamaji:USB_A" H 10450 4560 50  0001 C CNN
 F 3 "" H 10450 4560 50  0001 C CNN
 	1    10300 4610
