File: pcb/v3/kamaji.sch (KiCad schematic (older format))
At the start: 38 parts

Commit message: finish the v3 schematic and map most of the footprints
Parts:
- added J1: UART, Pin_Headers:Pin_Header_Straight_1x06_Pitch2.54mm, symbol UART_6pin
- added RV2: POT, Potentiometers:Potentiometer_Triwood_RM-065, symbol POT
- added U2: BOOST_24V, symbol BOOST_24V
- C1, C2, C5: renamed from C?; footprint (none) -> Capacitors_THT:C_Disc_D3.8mm_W2.6mm_P2.50mm
- C3, C4: renamed from C?; footprint (none) -> Capacitors_SMD:C_1206_HandSoldering
- F1: renamed from F?; footprint (none) -> Capacitors_THT:C_Disc_D5.0mm_W2.5mm_P5.00mm
- J10: renamed from J?; footprint (none) -> kamaji:USB_A
- J2: renamed from J?; footprint (none) -> Pin_Headers:Pin_Header_Straight_2x05_Pitch2.54mm
- J3, J4, J5, J6, J7, J8: renamed from J?; footprint (none) -> kamaji:RJ10
- J9: renamed from J?; footprint (none) -> kamaji:USB_B
- JP1: renamed from JP?; value 24V -> 5V; footprint (none) -> Pin_Headers:Pin_Header_Straight_1x02_Pitch2.54mm
- JP2: renamed from JP?; value 5V -> 24V; footprint (none) -> Pin_Headers:Pin_Header_Straight_1x02_Pitch2.54mm
- LS1: renamed from LS?; footprint (none) -> kamaji:Buzzer_ARIO_98dB
- Q1: renamed from Q?; footprint TO_SOT_Packages_THT:TO-92_Molded_Narrow -> TO_SOT_Packages_THT:TO-92_Inline_Narrow_Oval
- Q2: renamed from Q?; footprint TO_SOT_Packages_THT:TO-220_Vertical -> TO_SOT_Packages_THT:TO-220-3_Horizontal
- R1, R10, R2, R3, R4, R5, R6, R7, R8, R9: renamed from R?; footprint (none) -> Resistors_THT:R_Axial_DIN0207_L6.3mm_D2.5mm_P10.16mm_Horizontal
- RV1: renamed from RV?; footprint (none) -> kamaji:Potentiometer_Wheel_16mm
- SW1, SW2, SW3: renamed from SW?; footprint (none) -> Buttons_Switches_THT:SW_PUSH-12mm_Wuerth-430476085716
- U1: renamed from U?; footprint DIL40 -> Housings_DIP:DIP-40_W15.24mm_LongPads
- Y1: renamed from Y?; footprint (none) -> Crystals:Crystal_HC49-U_Vertical
- gave numbers to parts that had none: 2
Connections:
- net labels added: MC_RX, MC_TX
- net labels removed: +24V
- wire segments 70 -> 72
- no-connect marks 11 -> 14
Other:
- note removed: "TODO: Boost converter"
- note removed: "TODO: UART header"

Commit message: add 2004A LCD footprint
Parts:
- DS1: footprint Displays:WC1602A -> kamaji:LCD2004
- U2: footprint (none) -> Pin_Headers:Pin_Header_Straight_1x05_Pitch2.54mm
Other:
- note added: "TODO: Replace boost converter footprint"
Changed lines of the file:
@@
 F 0 "DS1" H 4935 2575 50  0000 C CNN
 F 1 "WC1602A" H 5375 2575 50  0000 C CNN
-F 2 "Displays:WC1602A" H 5165 925 50  0001 C CIN
+F 2 "kamaji:LCD2004" H 5165 925 50  0001 C CIN
 F 3 "" H 5865 1825 50  0001 C CNN
 	1    5165 1825
@@
 F 0 "U2" H 7600 1770 60  0000 C CNN
 F 1 "BOOST_24V" H 7600 2070 60  0000 C CNN
-F 2 "" H 7600 1770 60  0001 C CNN
+F 2 "Pin_Headers:Pin_Header_Straight_1x05_Pitch2.54mm" H 7600 1770 60  0001 C CNN
 F 3 "" H 7600 1770 60  0001 C CNN
 	1    7600 1770
@@
 	1    0    0    -1
 $EndComp
+Text Notes 7295 6830 0    79   Italic 0
+TODO: Replace boost converter footprint
 $EndSCHEMATC

Commit message: change screen and buttons footprints
Parts:
- SW1, SW2, SW3: footprint Buttons_Switches_THT:SW_PUSH-12mm_Wuerth-430476085716 -> kamaji:Pushbutton_12mm
Changed lines of the file:
@@
 F 0 "SW1" H 7115 4345 50  0000 L CNN
 F 1 "SW_Push" H 7065 4185 50  0001 C CNN
-F 2 "Buttons_Switches_THT:SW_PUSH-12mm_Wuerth-430476085716" H 7065 4445 50  0001 C CNN
+F 2 "kamaji:Pushbutton_12mm" H 7065 4445 50  0001 C CNN
 F 3 "" H 7065 4445 50  0001 C CNN
 	1    7065 4245
@@
 F 0 "SW2" H 7115 4775 50  0000 L CNN
 F 1 "SW_Push" H 7065 4615 50  0001 C CNN
-F 2 "Buttons_Switches_THT:SW_PUSH-12mm_Wuerth-430476085716" H 7065 4875 50  0001 C CNN
+F 2 "kamaji:Pushbutton_12mm" H 7065 4875 50  0001 C CNN
 F 3 "" H 7065 4875 50  0001 C CNN
 	1    7065 4675
@@
 F 0 "SW3" H 7120 5220 50  0000 L CNN
 F 1 "SW_Push" H 7070 5060 50  0001 C CNN
-F 2 "Buttons_Switches_THT:SW_PUSH-12mm_Wuerth-430476085716" H 7070 5320 50  0001 C CNN
+F 2 "kamaji:Pushbutton_12mm" H 7070 5320 50  0001 C CNN
 F 3 "" H 7070 5320 50  0001 C CNN
 	1    7070 5120

Commit message: mostly finish the v3 layout
Parts:
- removed RN1: 10K, Resistors_THT:R_Array_SIP9, symbol R_Network08
- added JP3: UART_PWR, Pin_Headers:Pin_Header_Straight_1x02_Pitch2.54mm, symbol Jumper_NC_Small
- J1: value UART -> UART_6pin; footprint Pin_Headers:Pin_Header_Straight_1x06_Pitch2.54mm -> kamaji:Pin_Header_Angled_1x06_Pitch2.54mm
- Q2: footprint TO_SOT_Packages_THT:TO-220-3_Horizontal -> kamaji:TO-220-3_Horizontal
Connections:
- net labels added: AVR_RX, AVR_TX, LCD_D4, LCD_D5, LCD_D6, LCD_D7, LCD_EN, LCD_RS
- net labels removed: MC_RX, MC_TX
- wire segments 72 -> 42
- no-connect marks 14 -> 12
Other:
- note added: "LCD SCREEN"
- note added: "UART\nCONNECTOR"

Commit message: v3 PCB: final touches
Parts:
- C3, C4: footprint Capacitors_SMD:C_1206_HandSoldering -> Capacitors_THT:C_Disc_D3.8mm_W2.6mm_P2.50mm
Changed lines of the file:
@@
 F 0 "C3" H 905 2400 50  0000 L CNN
 F 1 "22pF" H 905 2200 50  0000 L CNN
-F 2 "Capacitors_SMD:C_1206_HandSoldering" H 918 2150 50  0001 C CNN
+F 2 "Capacitors_THT:C_Disc_D3.8mm_W2.6mm_P2.50mm" H 918 2150 50  0001 C CNN
 F 3 "" H 880 2300 50  0001 C CNN
 	1    880  2300
@@
 F 0 "C4" H 905 2800 50  0000 L CNN
 F 1 "22pF" H 905 2600 50  0000 L CNN
-F 2 "Capacitors_SMD:C_1206_HandSoldering" H 918 2550 50  0001 C CNN
+F 2 "Capacitors_THT:C_Disc_D3.8mm_W2.6mm_P2.50mm" H 918 2550 50  0001 C CNN
 F 3 "" H 880 2700 50  0001 C CNN
 	1    880  2700
