File: pcb/v3/v3.sch (KiCad schematic (older format))
At the start: 34 parts

Commit message: finish v3 schematic
Parts:
- added C1, C4, C5: 0.1uF, symbol Device:C
- added C6: 20uF, symbol Device:C
- added J10: USB_A, symbol Connector:USB_A
- added J9: USB_B, symbol Connector:USB_B
- added Q1, Q3: BS170, Package_TO_SOT_THT:TO-92_Inline, symbol Transistor_FET:BS170
- added R11, R18: 1K, symbol Device:R
- added R13, R19: 10K, symbol Device:R
- added R14, R15, R16, R17: 200R, symbol Device:R
- gave numbers to parts that had none: 34
Connections:
- wire segments 47 -> 59
- no-connect marks 5 -> 8
Other:
- note removed: "TODO: Lamp\nTODO: Dummy load\nTODO: Power connector\nTODO: Bypass capacitors"
- moved on the sheet: C2, C3, J2, J8, JP1, JP2, LS1, Q2, R12, RV2, SW1, SW2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

Commit message: v3: draw missing footprints, start layout
Parts:
- C1, C2, C3, C4, C5, C6: footprint (none) -> Capacitor_THT:C_Disc_D3.8mm_W2.6mm_P2.50mm
- J1, J3, J4, J5, J6, J7: footprint (none) -> kamaji:RJ10
- J10: footprint (none) -> kamaji:USB_A
- J2: footprint (none) -> kamaji:ATmega_ISP_6pin
- J8: footprint (none) -> kamaji:DD1718PA
- J9: footprint (none) -> kamaji:USB_B
- JP1, JP2: footprint (none) -> Connector_PinHeader_2.54mm:PinHeader_1x02_P2.54mm_Vertical
- LS1: footprint (none) -> kamaji:Buzzer_ARIO_98dB
- R1, R10, R11, R12, R13, R14, R15, R16, R17, R18, R19, R2, R3, R4, R5, R6, R7, R8, R9: footprint (none) -> Resistor_THT:R_Axial_DIN0207_L6.3mm_D2.5mm_P10.16mm_Horizontal
- RV1: footprint (none) -> Potentiometer_THT:Potentiometer_Vishay_T73YP_Vertical
- RV2: value R_POT -> VOLUME; footprint (none) -> kamaji:Potentiometer_Wheel_16mm
- SW1, SW2, SW3: footprint (none) -> kamaji:Pushbutton_12mm
- U2: footprint (none) -> Package_DIP:DIP-16_W7.62mm_LongPads
- U3: footprint Display:RC1602A -> kamaji:LCD2004
- Y1: footprint (none) -> Crystal:Crystal_HC49-U_Vertical

Commit message: v3: initial component placement
Parts:
- removed J2: ICSP, kamaji:ATmega_ISP_6pin, symbol Connector_Generic:Conn_02x03_Odd_Even
- added J2: ICSP, Connector_IDC:IDC-Header_2x05_P2.54mm_Horizontal, symbol Connector_Generic:Conn_02x05_Odd_Even
- C1, C2, C3, C4, C5, C6: footprint Capacitor_THT:C_Disc_D3.8mm_W2.6mm_P2.50mm -> Capacitor_SMD:C_1206_3216Metric_Pad1.42x1.75mm_HandSolder
- R1, R10, R11, R12, R13, R18, R19, R2, R3, R5, R6, R7, R8, R9: footprint Resistor_THT:R_Axial_DIN0207_L6.3mm_D2.5mm_P10.16mm_Horizontal -> Resistor_SMD:R_1206_3216Metric_Pad1.42x1.75mm_HandSolder
Connections:
- wire segments 59 -> 62
- no-connect marks 8 -> 9
Changed lines of the file:
@@
 F 0 "C2" V 1148 3440 50  0000 C CNN
 F 1 "20pF" V 1239 3440 50  0000 C CNN
-F 2 "Capacitor_THT:C_Disc_D3.8mm_W2.6mm_P2.50mm" H 1438 3290 50  0001 C CNN
+F 2 "Capacitor_SMD:C_1206_3216Metric_Pad1.42x1.75mm_HandSolder" H 1438 3290 50  0001 C CNN
 F 3 "~" H 1400 3440 50  0001 C CNN
 	1    1400 3440
@@
 F 0 "C3" V 1620 3740 50  0000 C CNN
 F 1 "20pF" V 1530 3740 50  0000 C CNN
-F 2 "Capacitor_THT:C_Disc_D3.8mm_W2.6mm_P2.50mm" H 1438 3590 50  0001 C CNN
+F 2 "Capacitor_SMD:C_1206_3216Metric_Pad1.42x1.75mm_HandSolder" H 1438 3590 50  0001 C CNN
 F 3 "~" H 1400 3740 50  0001 C CNN
 	1    1400 3740
@@
 $EndComp
 $Comp
-L Connector_Generic:Conn_02x03_Odd_Even J2
-U 1 1 5C559237
-P 1200 2410
-F 0 "J2" H 1250 2727 50  0000 C CNN
-F 1 "ICSP" H 1250 2636 50  0000 C CNN
-F 2 "kamaji:ATmega_ISP_6pin" H 1200 2410 50  0001 C CNN
-F 3 "~" H 1200 2410 50  0001 C CNN
-	1    1200 2410
-	1    0    0    -1
-$EndComp
-$Comp
 L power:VCC #PWR0107
 U 1 1 5C559384
-P 1500 2310
-F 0 "#PWR0107" H 1500 2160 50  0001 C CNN
-F 1 "VCC" H 1580 2450 50  0000 C CNN
-F 2 "" H 1500 2310 50  0001 C CNN
-F 3 "" H 1500 2310 50  0001 C CNN
-	1    1500 2310
+P 1460 2110
+F 0 "#PWR0107" H 1460 1960 50  0001 C CNN
+F 1 "VCC" H 1540 2250 50  0000 C CNN
+F 2 "" H 1460 2110 50  0001 C CNN
+F 3 "" H 1460 2110 50  0001 C CNN
+	1    1460 2110
 	1    0    0    -1
 $EndComp
@@
 L power:GND #PWR0108
 U 1 1 5C5594C3
-P 1500 2510
-F 0 "#PWR0108" H 1500 2260 50  0001 C CNN
-F 1 "GND" H 1500 2360 50  0000 C CNN
-F 2 "" H 1500 2510 50  0001 C CNN
-F 3 "" H 1500 2510 50  0001 C CNN
-	1    1500 2510
-	1    0    0    -1
-$EndComp
-Text Label 1500 2410 0    50   ~ 0
+P 1460 2510
+F 0 "#PWR0108" H 1460 2260 50  0001 C CNN
+F 1 "GND" H 1460 2360 50  0000 C CNN
+F 2 "" H 1460 2510 50  0001 C CNN
+F 3 "" H 1460 2510 50  0001 C CNN
+	1    1460 2510
+	1    0    0    -1
+$EndComp
+Text Label 960  2110 2    50   ~ 0
 MOSI
-Text Label 1000 2310 2    50   ~ 0
+Text Label 960  2510 2    50   ~ 0
 MISO
-Text Label 1000 2410 2    50   ~ 0
+Text Label 960  2410 2    50   ~ 0
 SCK
-Text Label 1000 2510 2    50   ~ 0
+Text Label 960  2310 2    50   ~ 0
 RST
 $Comp
@@
 F 0 "R1" V 1040 7450 50  0000 L CNN
 F 1 "1K" V 940 7400 50  0000 L CNN
-F 2 "Resistor_THT:R_Axial_DIN0207_L6.3mm_D2.5mm_P10.16mm_Horizontal" V 870 7450 50  0001 C CNN
+F 2 "Resistor_SMD:R_1206_3216Metric_Pad1.42x1.75mm_HandSolder" V 870 7450 50  0001 C CNN
 F 3 "~" H 940 7450 50  0001 C CNN
 	1    940  7450
@@
 F 0 "R2" V 2020 7450 50  0000 L CNN
 F 1 "1K" V 1920 7400 50  0000 L CNN
-F 2 "Resistor_THT:R_Axial_DIN0207_L6.3mm_D2.5mm_P10.16mm_Horizontal" V 1850 7450 50  0001 C CNN
+F 2 "Resistor_SMD:R_1206_3216Metric_Pad1.42x1.75mm_HandSolder" V 1850 7450 50  0001 C CNN
 F 3 "~" H 1920 7450 50  0001 C CNN
 	1    1920 7450
@@
 F 0 "R3" V 2970 7450 50  0000 L CNN
 F 1 "1K" V 2870 7400 50  0000 L CNN
-F 2 "Resistor_THT:R_Axial_DIN0207_L6.3mm_D2.5mm_P10.16mm_Horizontal" V 2800 7450 50  0001 C CNN
+F 2 "Resistor_SMD:R_1206_3216Metric_Pad1.42x1.75mm_HandSolder" V 2800 7450 50  0001 C CNN
 F 3 "~" H 2870 7450 50  0001 C CNN
 	1    2870 7450
@@
 F 0 "R5" V 3920 7440 50  0000 L CNN
 F 1 "1K" V 3820 7390 50  0000 L CNN
-F 2 "Resistor_THT:R_Axial_DIN0207_L6.3mm_D2.5mm_P10.16mm_Horizontal" V 3750 7440 50  0001 C CNN
+F 2 "Resistor_SMD:R_1206_3216Metric_Pad1.42x1.75mm_HandSolder" V 3750 7440 50  0001 C CNN
 F 3 "~" H 3820 7440 50  0001 C CNN
 	1    3820 7440
@@
 F 0 "R8" V 4910 7460 50  0000 L CNN
 F 1 "1K" V 4810 7410 50  0000 L CNN
-F 2 "Resistor_THT:R_Axial_DIN0207_L6.3mm_D2.5mm_P10.16mm_Horizontal" V 4740 7460 50  0001 C CNN
+F 2 "Resistor_SMD:R_1206_3216Metric_Pad1.42x1.75mm_HandSolder" V 4740 7460 50  0001 C CNN
 F 3 "~" H 4810 7460 50  0001 C CNN
 	1    4810 7460
@@
 F 0 "R7" H 4720 1080 50  0000 L CNN
 F 1 "4K7" V 4670 1010 50  0000 L CNN
-F 2 "Resistor_THT:R_Axial_DIN0207_L6.3mm_D2.5mm_P10.16mm_Horizontal" V 4600 1080 50  0001 C CNN
+F 2 "Resistor_SMD:R_1206_3216Metric_Pad1.42x1.75mm_HandSolder" V 4600 1080 50  0001 C CNN
 F 3 "~" H 4670 1080 50  0001 C CNN
 	1    4670 1080
@@
 F 0 "R6" H 4480 1070 50  0000 L CNN
 F 1 "4K7" V 4430 1000 50  0000 L CNN
-F 2 "Resistor_THT:R_Axial_DIN0207_L6.3mm_D2.5mm_P10.16mm_Horizontal" V 4360 1070 50  0001 C CNN
+F 2 "Resistor_SMD:R_1206_3216Metric_Pad1.42x1.75mm_HandSolder" V 4360 1070 50  0001 C CNN
 F 3 "~" H 4430 1070 50  0001 C CNN
 	1    4430 1070
@@
 F 0 "R10" V 5810 4050 50  0000 C CNN
 F 1 "1K" V 5910 4050 50  0000 C CNN
-F 2 "Resistor_THT:R_Axial_DIN0207_L6.3mm_D2.5mm_P10.16mm_Horizontal" V 5840 4050 50  0001 C CNN
+F 2 "Resistor_SMD:R_1206_3216Metric_Pad1.42x1.75mm_HandSolder" V 5840 4050 50  0001 C CNN
 F 3 "~" H 5910 4050 50  0001 C CNN
 	1    5910 4050
@@
 F 0 "R9" V 5920 7480 50  0000 L CNN
 F 1 "1K" V 5820 7430 50  0000 L CNN
-F 2 "Resistor_THT:R_Axial_DIN0207_L6.3mm_D2.5mm_P10.16mm_Horizontal" V 5750 7480 50  0001 C CNN
+F 2 "Resistor_SMD:R_1206_3216Metric_Pad1.42x1.75mm_HandSolder" V 5750 7480 50  0001 C CNN
 F 3 "~" H 5820 7480 50  0001 C CNN
 	1    5820 7480
@@
 F 0 "R12" V 7560 3880 50  0000 C CNN
 F 1 "1K" V 7660 3880 50  0000 C CNN
-F 2 "Resistor_THT:R_Axial_DIN0207_L6.3mm_D2.5mm_P10.16mm_Horizontal" V 7590 3880 50  0001 C CNN
+F 2 "Resistor_SMD:R_1206_3216Metric_Pad1.42x1.75mm_HandSolder" V 7590 3880 50  0001 C CNN
 F 3 "~" H 7660 3880 50  0001 C CNN
 	1    7660 3880
@@
 F 0 "R19" H 9700 3950 50  0000 L CNN
 F 1 "10K" V 9870 3880 50  0000 L CNN
-F 2 "Resistor_THT:R_Axial_DIN0207_L6.3mm_D2.5mm_P10.16mm_Horizontal" V 9800 3960 50  0001 C CNN
+F 2 "Resistor_SMD:R_1206_3216Metric_Pad1.42x1.75mm_HandSolder" V 9800 3960 50  0001 C CNN
 F 3 "~" H 9870 3960 50  0001 C CNN
 	1    9870 3960
@@
 F 0 "R18" V 9500 3820 50  0000 C CNN
 F 1 "1K" V 9590 3810 50  0000 C CNN
-F 2 "Resistor_THT:R_Axial_DIN0207_L6.3mm_D2.5mm_P10.16mm_Horizontal" V 9520 3810 50  0001 C CNN
+F 2 "Resistor_SMD:R_1206_3216Metric_Pad1.42x1.75mm_HandSolder" V 9520 3810 50  0001 C CNN
 F 3 "~" H 9590 3810 50  0001 C CNN
 	1    9590 3810
@@
 F 0 "R13" H 7540 5480 50  0000 L CNN
 F 1 "10K" V 7710 5410 50  0000 L CNN
-F 2 "Resistor_THT:R_Axial_DIN0207_L6.3mm_D2.5mm_P10.16mm_Horizontal" V 7640 5490 50  0001 C CNN
+F 2 "Resistor_SMD:R_1206_3216Metric_Pad1.42x1.75mm_HandSolder" V 7640 5490 50  0001 C CNN
 F 3 "~" H 7710 5490 50  0001 C CNN
 	1    7710 5490
@@
 F 0 "R11" V 7390 5350 50  0000 C CNN
 F 1 "1K" V 7480 5340 50  0000 C CNN
-F 2 "Resistor_THT:R_Axial_DIN0207_L6.3mm_D2.5mm_P10.16mm_Horizontal" V 7410 5340 50  0001 C CNN
+F 2 "Resistor_SMD:R_1206_3216Metric_Pad1.42x1.75mm_HandSolder" V 7410 5340 50  0001 C CNN
 F 3 "~" H 7480 5340 50  0001 C CNN
 	1    7480 5340
@@
 F 0 "C1" H 1405 1176 50  0000 L CNN
 F 1 "0.1uF" H 1405 1085 50  0000 L CNN
-F 2 "Capacitor_THT:C_Disc_D3.8mm_W2.6mm_P2.50mm" H 1328 980 50  0001 C CNN
+F 2 "Capacitor_SMD:C_1206_3216Metric_Pad1.42x1.75mm_HandSolder" H 1328 980 50  0001 C CNN
 F 3 "~" H 1290 1130 50  0001 C CNN
 	1    1290 1130
@@
 F 0 "C5" H 6225 2226 50  0000 L CNN
 F 1 "0.1uF" H 6225 2135 50  0000 L CNN
-F 2 "Capacitor_THT:C_Disc_D3.8mm_W2.6mm_P2.50mm" H 6148 2030 50  0001 C CNN
+F 2 "Capacitor_SMD:C_1206_3216Metric_Pad1.42x1.75mm_HandSolder" H 6148 2030 50  0001 C CNN
 F 3 "~" H 6110 2180 50  0001 C CNN
 	1    6110 2180
@@
 F 0 "C4" H 6015 4716 50  0000 L CNN
 F 1 "0.1uF" H 6015 4625 50  0000 L CNN
-F 2 "Capacitor_THT:C_Disc_D3.8mm_W2.6mm_P2.50mm" H 5938 4520 50  0001 C CNN
+F 2 "Capacitor_SMD:C_1206_3216Metric_Pad1.42x1.75mm_HandSolder" H 5938 4520 50  0001 C CNN
 F 3 "~" H 5900 4670 50  0001 C CNN
 	1    5900 4670
@@
 F 0 "C6" H 8725 1566 50  0000 L CNN
 F 1 "20uF" H 8725 1475 50  0000 L CNN
-F 2 "Capacitor_THT:C_Disc_D3.8mm_W2.6mm_P2.50mm" H 8648 1370 50  0001 C CNN
+F 2 "Capacitor_SMD:C_1206_3216Metric_Pad1.42x1.75mm_HandSolder" H 8648 1370 50  0001 C CNN
 F 3 "~" H 8610 1520 50  0001 C CNN
 	1    8610 1520
@@
 Text Label 3250 2650 0    50   ~ 0
 LCD3
+$Comp
+L Connector_Generic:Conn_02x05_Odd_Even J2
+U 1 1 5C5C4D22
+P 1160 2310
+F 0 "J2" H 1210 2727 50  0000 C CNN
+F 1 "ICSP" H 1210 2636 50  0000 C CNN
+F 2 "Connector_IDC:IDC-Header_2x05_P2.54mm_Horizontal" H 1160 2310 50  0001 C CNN
+F 3 "~" H 1160 2310 50  0001 C CNN
+	1    1160 2310
+	1    0    0    -1
+$EndComp
+Wire Wire Line
+	1460 2510 1460 2410
+Connection ~ 1460 2510
+Connection ~ 1460 2310
+Wire Wire Line
+	1460 2310 1460 2210
+Connection ~ 1460 2410
+Wire Wire Line
+	1460 2410 1460 2310
+NoConn ~ 960  2210
 $EndSCHEMATC

Commit message: v3: move components around
Parts:
- added C7: 0.1uF, Capacitor_SMD:C_1206_3216Metric_Pad1.42x1.75mm_HandSolder, symbol Device:C
- R4: footprint Resistor_THT:R_Axial_DIN0207_L6.3mm_D2.5mm_P10.16mm_Horizontal -> Resistor_SMD:R_1206_3216Metric_Pad1.42x1.75mm_HandSolder
Changed lines of the file:
@@
 F 0 "R4" H 3760 2846 50  0000 L CNN
 F 1 "10K" H 3760 2755 50  0000 L CNN
-F 2 "Resistor_THT:R_Axial_DIN0207_L6.3mm_D2.5mm_P10.16mm_Horizontal" V 3620 2800 50  0001 C CNN
+F 2 "Resistor_SMD:R_1206_3216Metric_Pad1.42x1.75mm_HandSolder" V 3620 2800 50  0001 C CNN
 F 3 "~" H 3690 2800 50  0001 C CNN
 	1    3690 2800
@@
 Wire Wire Line
 	5160 7200 5220 7200
-Text Label 3460 1750 0    50   ~ 0
+Text Label 3460 1950 0    50   ~ 0
 CBTN1
 $Comp
@@
 Text Label 3460 1850 0    50   ~ 0
 CBTN2
-Text Label 3460 1950 0    50   ~ 0
+Text Label 3460 1750 0    50   ~ 0
 CBTN3
 Text Label 3250 2050 0    50   ~ 0
@@
 Text Label 5860 1730 0    50   ~ 0
 PLED6
+Text Label 3250 3650 0    50   ~ 0
+PBTN1
+Text Label 3250 3550 0    50   ~ 0
+PBTN2
+Text Label 3250 3450 0    50   ~ 0
+PBTN3
+Text Label 3250 3350 0    50   ~ 0
+PBTN4
+Text Label 3250 3250 0    50   ~ 0
+PBTN5
 Text Label 3250 3150 0    50   ~ 0
-PBTN1
-Text Label 3250 3250 0    50   ~ 0
-PBTN2
-Text Label 3250 3350 0    50   ~ 0
-PBTN3
-Text Label 3250 3450 0    50   ~ 0
-PBTN4
-Text Label 3250 3550 0    50   ~ 0
-PBTN5
-Text Label 3250 3650 0    50   ~ 0
 PBTN6
 $Comp
@@
 	1460 2410 1460 2310
 NoConn ~ 960  2210
+$Comp
+L Device:C C7
+U 1 1 5C5DFDB3
+P 730 1120
+F 0 "C7" H 845 1166 50  0000 L CNN
+F 1 "0.1uF" H 845 1075 50  0000 L CNN
+F 2 "Capacitor_SMD:C_1206_3216Metric_Pad1.42x1.75mm_HandSolder" H 768 970 50  0001 C CNN
+F 3 "~" H 730 1120 50  0001 C CNN
+	1    730  1120
+	1    0    0    -1
+$EndComp
+$Comp
+L power:GND #PWR02
+U 1 1 5C5DFDBA
+P 730 1270
+F 0 "#PWR02" H 730 1020 50  0001 C CNN
+F 1 "GND" H 735 1097 50  0000 C CNN
+F 2 "" H 730 1270 50  0001 C CNN
+F 3 "" H 730 1270 50  0001 C CNN
+	1    730  1270
+	1    0    0    -1
+$EndComp
+$Comp
+L power:VCC #PWR01
+U 1 1 5C5DFDC0
+P 730 970
+F 0 "#PWR01" H 730 820 50  0001 C CNN
+F 1 "VCC" H 747 1143 50  0000 C CNN
+F 2 "" H 730 970 50  0001 C CNN
+F 3 "" H 730 970 50  0001 C CNN
+	1    730  970
+	1    0    0    -1
+$EndComp
 $EndSCHEMATC

Commit message: v3: finish layout
Parts:
- Q1, Q2, Q3: footprint Package_TO_SOT_THT:TO-92_Inline -> Package_TO_SOT_THT:TO-92_Inline_Wide
Changed lines of the file:
@@
 Wire Wire Line
 	5160 7200 5220 7200
-Text Label 3460 1950 0    50   ~ 0
+Text Label 3460 1750 0    50   ~ 0
 CBTN1
 $Comp
@@
 Wire Wire Line
 	1050 3440 1250 3440
+Text Label 3460 1950 0    50   ~ 0
+CBTN2
 Text Label 3460 1850 0    50   ~ 0
-CBTN2
-Text Label 3460 1750 0    50   ~ 0
 CBTN3
 Text Label 3250 2050 0    50   ~ 0
@@
 F 0 "Q2" H 8201 3926 50  0000 L CNN
 F 1 "2N3904" H 8201 3835 50  0000 L CNN
-F 2 "Package_TO_SOT_THT:TO-92_Inline" H 8210 3805 50  0001 L CIN
+F 2 "Package_TO_SOT_THT:TO-92_Inline_Wide" H 8210 3805 50  0001 L CIN
 F 3 "https://www.fairchildsemi.com/datasheets/2N/2N3904.pdf" H 8010 3880 50  0001 L CNN
 	1    8010 3880
@@
 Text Label 7510 3880 2    50   ~ 0
 SPK
+Text Label 3250 3850 0    50   ~ 0
+LCDRS
 Text Label 3250 3750 0    50   ~ 0
-LCDRS
-Text Label 3250 3850 0    50   ~ 0
 LCDE
 Text Label 3250 1650 0    50   ~ 0
@@
 F 0 "Q3" H 10275 3856 50  0000 L CNN
 F 1 "BS170" H 10275 3765 50  0000 L CNN
-F 2 "Package_TO_SOT_THT:TO-92_Inline" H 10270 3735 50  0001 L CIN
+F 2 "Package_TO_SOT_THT:TO-92_Inline_Wide" H 10270 3735 50  0001 L CIN
 F 3 "http://www.fairchildsemi.com/ds/BS/BS170.pdf" H 10070 3810 50  0001 L CNN
 	1    10070 3810
@@
 F 0 "Q1" H 8115 5386 50  0000 L CNN
 F 1 "BS170" H 8115 5295 50  0000 L CNN
-F 2 "Package_TO_SOT_THT:TO-92_Inline" H 8110 5265 50  0001 L CIN
+F 2 "Package_TO_SOT_THT:TO-92_Inline_Wide" H 8110 5265 50  0001 L CIN
 F 3 "http://www.fairchildsemi.com/ds/BS/BS170.pdf" H 7910 5340 50  0001 L CNN
 	1    7910 5340

Commit message: v3.1 schematic
Parts:
- removed Q1: BS170, Package_TO_SOT_THT:TO-92_Inline_Wide, symbol Transistor_FET:BS170
- removed R11: 1K, Resistor_SMD:R_1206_3216Metric_Pad1.42x1.75mm_HandSolder, symbol Device:R
- removed R13: 10K, Resistor_SMD:R_1206_3216Metric_Pad1.42x1.75mm_HandSolder, symbol Device:R
- removed R14, R15, R16, R17: 200R, Resistor_THT:R_Axial_DIN0207_L6.3mm_D2.5mm_P10.16mm_Horizontal, symbol Device:R
Connections:
- net labels removed: LOAD
- wire segments 62 -> 54
- no-connect marks 9 -> 10
Other:
- moved on the sheet: LS1, Q2, R12, RV2
Changed lines of the file:
@@
 EESchema Schematic File Version 4
 LIBS:v3-cache
-EELAYER 26 0
+EELAYER 29 0
 EELAYER END
 $Descr A4 11693 8268
@@
 F 3 "~" H 7630 3410 50  0001 C CNN
 	1    7630 3410
-	1    0    0    -1
+	-1   0    0    1
 $EndComp
 $Comp
@@
 L Device:Speaker_Crystal LS1
 U 1 1 5C5A8DB6
-P 8310 3410
-F 0 "LS1" H 8485 3406 50  0000 L CNN
-F 1 "Speaker" H 8485 3315 50  0000 L CNN
-F 2 "kamaji:Buzzer_ARIO_98dB" H 8275 3360 50  0001 C CNN
-F 3 "~" H 8275 3360 50  0001 C CNN
-	1    8310 3410
-	1    0    0    -1
-$EndComp
-Wire Wire Line
-	7780 3410 8110 3410
+P 7280 3510
+F 0 "LS1" H 7455 3506 50  0000 L CNN
+F 1 "Speaker" H 7455 3415 50  0000 L CNN
+F 2 "kamaji:Buzzer_ARIO_98dB" H 7245 3460 50  0001 C CNN
+F 3 "~" H 7245 3460 50  0001 C CNN
+	1    7280 3510
+	-1   0    0    1
+$EndComp
 $Comp
 L Transistor_BJT:2N3904 Q2
 U 1 1 5C5AA536
-P 8010 3880
-F 0 "Q2" H 8201 3926 50  0000 L CNN
-F 1 "2N3904" H 8201 3835 50  0000 L CNN
-F 2 "Package_TO_SOT_THT:TO-92_Inline_Wide" H 8210 3805 50  0001 L CIN
-F 3 "https://www.fairchildsemi.com/datasheets/2N/2N3904.pdf" H 8010 3880 50  0001 L CNN
-	1    8010 3880
-	1    0    0    -1
-$EndComp
-Wire Wire Line
-	8110 3510 8110 3680
+P 7380 3940
+F 0 "Q2" H 7571 3986 50  0000 L CNN
+F 1 "2N3904" H 7571 3895 50  0000 L CNN
+F 2 "Package_TO_SOT_THT:TO-92_Inline_Wide" H 7580 3865 50  0001 L CIN
+F 3 "https://www.fairchildsemi.com/datasheets/2N/2N3904.pdf" H 7380 3940 50  0001 L CNN
+	1    7380 3940
+	1    0    0    -1
+$EndComp
 $Comp
 L power:GND #PWR0145
 U 1 1 5C5ABB73
-P 8110 4080
-F 0 "#PWR0145" H 8110 3830 50  0001 C CNN
-F 1 "GND" H 8110 3910 50  0000 C CNN
-F 2 "" H 8110 4080 50  0001 C CNN
-F 3 "" H 8110 4080 50  0001 C CNN
-	1    8110 4080
+P 7480 4140
+F 0 "#PWR0145" H 7480 3890 50  0001 C CNN
+F 1 "GND" H 7480 3970 50  0000 C CNN
+F 2 "" H 7480 4140 50  0001 C CNN
+F 3 "" H 7480 4140 50  0001 C CNN
+	1    7480 4140
 	1    0    0    -1
 $EndComp
@@
 L Device:R R12
 U 1 1 5C5ADC70
-P 7660 3880
-F 0 "R12" V 7560 3880 50  0000 C CNN
-F 1 "1K" V 7660 3880 50  0000 C CNN
-F 2 "Resistor_SMD:R_1206_3216Metric_Pad1.42x1.75mm_HandSolder" V 7590 3880 50  0001 C CNN
-F 3 "~" H 7660 3880 50  0001 C CNN
-	1    7660 3880
+P 7030 3940
+F 0 "R12" V 6930 3940 50  0000 C CNN
+F 1 "1K" V 7030 3940 50  0000 C CNN
+F 2 "Resistor_SMD:R_1206_3216Metric_Pad1.42x1.75mm_HandSolder" V 6960 3940 50  0001 C CNN
+F 3 "~" H 7030 3940 50  0001 C CNN
+	1    7030 3940
 	0    -1   -1   0
 $EndComp
-Text Label 7510 3880 2    50   ~ 0
+Text Label 6880 3940 2    50   ~ 0
 SPK
 Text Label 3250 3850 0    50   ~ 0
@@
 Text Label 3250 3750 0    50   ~ 0
 LCDE
-Text Label 3250 1650 0    50   ~ 0
-LOAD
 $Comp
 L Connector:USB_A J10
@@
 	0    1    1    0
 $EndComp
-$Comp
-L Device:R R14
-U 1 1 5C584646
-P 8010 4990
-F 0 "R14" V 7920 4990 50  0000 C CNN
-F 1 "200R" V 8010 4990 50  0000 C CNN
-F 2 "Resistor_THT:R_Axial_DIN0207_L6.3mm_D2.5mm_P10.16mm_Horizontal" V 7940 4990 50  0001 C CNN
-F 3 "~" H 8010 4990 50  0001 C CNN
-	1    8010 4990
-	-1   0    0    1
-$EndComp
-$Comp
-L Device:R R15
-U 1 1 5C58600B
-P 8200 4990
-F 0 "R15" V 8110 4990 50  0000 C CNN
-F 1 "200R" V 8200 4990 50  0000 C CNN
-F 2 "Resistor_THT:R_Axial_DIN0207_L6.3mm_D2.5mm_P10.16mm_Horizontal" V 8130 4990 50  0001 C CNN
-F 3 "~" H 8200 4990 50  0001 C CNN
-	1    8200 4990
-	-1   0    0    1
-$EndComp
-$Comp
-L Device:R R16
-U 1 1 5C5861E8
-P 8410 4990
-F 0 "R16" V 8320 4990 50  0000 C CNN
-F 1 "200R" V 8410 4990 50  0000 C CNN
-F 2 "Resistor_THT:R_Axial_DIN0207_L6.3mm_D2.5mm_P10.16mm_Horizontal" V 8340 4990 50  0001 C CNN
-F 3 "~" H 8410 4990 50  0001 C CNN
-	1    8410 4990
-	-1   0    0    1
-$EndComp
-$Comp
-L Device:R R17
-U 1 1 5C58647C
-P 8610 4990
-F 0 "R17" V 8520 4990 50  0000 C CNN
-F 1 "200R" V 8610 4990 50  0000 C CNN
-F 2 "Resistor_THT:R_Axial_DIN0207_L6.3mm_D2.5mm_P10.16mm_Horizontal" V 8540 4990 50  0001 C CNN
-F 3 "~" H 8610 4990 50  0001 C CNN
-	1    8610 4990
-	-1   0    0    1
-$EndComp
-$Comp
-L power:VCC #PWR0153
-U 1 1 5C586CD2
-P 8010 4840
-F 0 "#PWR0153" H 8010 4690 50  0001 C CNN
-F 1 "VCC" H 8010 5010 50  0000 C CNN
-F 2 "" H 8010 4840 50  0001 C CNN
-F 3 "" H 8010 4840 50  0001 C CNN
-	1    8010 4840
-	1    0    0    -1
-$EndComp
-Wire Wire Line
-	8010 4840 8200 4840
-Connection ~ 8010 4840
-Wire Wire Line
-	8610 4840 8410 4840
-Wire Wire Line
-	8410 4840 8200 4840
-Connection ~ 8410 4840
-Connection ~ 8200 4840
-Wire Wire Line
-	8610 5140 8410 5140
-Connection ~ 8200 5140
-Wire Wire Line
-	8200 5140 8010 5140
-Connection ~ 8410 5140
-Wire Wire Line
-	8410 5140 8200 5140
-$Comp
-L Transistor_FET:BS170 Q1
-U 1 1 5C58B299
-P 7910 5340
-F 0 "Q1" H 8115 5386 50  0000 L CNN
-F 1 "BS170" H 8115 5295 50  0000 L CNN
-F 2 "Package_TO_SOT_THT:TO-92_Inline_Wide" H 8110 5265 50  0001 L CIN
-F 3 "http://www.fairchildsemi.com/ds/BS/BS170.pdf" H 7910 5340 50  0001 L CNN
-	1    7910 5340
-	1    0    0    -1
-$EndComp
-Connection ~ 8010 5140
-$Comp
-L power:GND #PWR0154
-U 1 1 5C58BB7F
-P 8010 5540
-F 0 "#PWR0154" H 8010 5290 50  0001 C CNN
-F 1 "GND" H 8010 5370 50  0000 C CNN
-F 2 "" H 8010 5540 50  0001 C CNN
-F 3 "" H 8010 5540 50  0001 C CNN
-	1    8010 5540
-	1    0    0    -1
-$EndComp
-$Comp
-L Device:R R13
-U 1 1 5C58D173
-P 7710 5490
-F 0 "R13" H 7540 5480 50  0000 L CNN
-F 1 "10K" V 7710 5410 50  0000 L CNN
-F 2 "Resistor_SMD:R_1206_3216Metric_Pad1.42x1.75mm_HandSolder" V 7640 5490 50  0001 C CNN
-F 3 "~" H 7710 5490 50  0001 C CNN
-	1    7710 5490
-	1    0    0    -1
-$EndComp
-$Comp
-L power:GND #PWR0155
-U 1 1 5C58D67E
-P 7710 5640
-F 0 "#PWR0155" H 7710 5390 50  0001 C CNN
-F 1 "GND" H 7710 5470 50  0000 C CNN
-F 2 "" H 7710 5640 50  0001 C CNN
-F 3 "" H 7710 5640 50  0001 C CNN
-	1    7710 5640
-	1    0    0    -1
-$EndComp
-$Comp
-L Device:R R11
-U 1 1 5C58DD91
-P 7480 5340
-F 0 "R11" V 7390 5350 50  0000 C CNN
-F 1 "1K" V 7480 5340 50  0000 C CNN
-F 2 "Resistor_SMD:R_1206_3216Metric_Pad1.42x1.75mm_HandSolder" V 7410 5340 50  0001 C CNN
-F 3 "~" H 7480 5340 50  0001 C CNN
-	1    7480 5340
-	0    1    1    0
-$EndComp
-Wire Wire Line
-	7630 5340 7710 5340
-Connection ~ 7710 5340
-Text Label 7330 5340 2    50   ~ 0
-LOAD
 $Comp
 L Device:C C1
@@
 	1    0    0    -1
 $EndComp
+Wire Wire Line
+	7480 3510 7480 3740
+NoConn ~ 3250 1650
 $EndSCHEMATC
