File: pcb/headless_v1/headless_v1.kicad_pcb (KiCad board)
At the start: 2 copper layers, 69 x 51 mm, 23 parts, among them J1 RJ10, J2 RJ10, J3 RJ10, J4 RJ10, J5 RJ10, J6 RJ10, J7 RJ10, J8 RJ10, SW1 RESET, U1 ProMicro

Commit message: Headless PCB v1.2
Parts:
- SW1: moved to B.Cu
- moved SW1 6.25 mm to (98.8, 72.0), turned to -90 degrees
Other:
- board text added: "Headless Kamaji v1.2 Ilya Strukov 2022 github.com/iley/kamaji"
- board text removed: "Headless Kamaji v1.1 Ilya Strukov 2022 github.com/iley/kamaji"

Commit message: Tweak a trace, cleanup
Other:
- outline, holes or cut-outs redrawn
Changed lines of the file:
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@@
     )
   )
-  (gr_rect (start 44.8 50) (end 113.8 101) (layer "Edge.Cuts") (width 0.1) (fill none))
+  (gr_line (start 114 51) (end 114 100) (layer "Edge.Cuts") (width 0.1))
+  (gr_arc (start 46 101) (mid 45.292893 100.707107) (end 45 100) (layer "Edge.Cuts") (width 0.1))
+  (gr_arc (start 114 100) (mid 113.707107 100.707107) (end 113 101) (layer "Edge.Cuts") (width 0.1))
+  (gr_line (start 45 100) (end 45 51) (layer "Edge.Cuts") (width 0.1))
+  (gr_arc (start 45 51) (mid 45.292893 50.292893) (end 46 50) (layer "Edge.Cuts") (width 0.1))
+  (gr_line (start 113 101) (end 46 101) (layer "Edge.Cuts") (width 0.1))
+  (gr_arc (start 113 50) (mid 113.707107 50.292893) (end 114 51) (layer "Edge.Cuts") (width 0.1))
+  (gr_line (start 46 50) (end 113 50) (layer "Edge.Cuts") (width 0.1))
   (gr_text "Headless Kamaji v1.2\nIlya Strukov 2022\ngithub.com/iley/kamaji" (at 66 75) (layer "B.SilkS")
     (effects (font (size 2 1.6) (thickness 0.25)) (justify mirror))
@@
   (arc (start 75.804139 86.494046) (mid 73.584486 86.120026) (end 71.528459 85.203784) (width 0.25) (layer "F.Cu") (net 7))
   (segment (start 100.51 93.46) (end 105.08 88) (width 0.25) (layer "F.Cu") (net 8))
-  (segment (start 76.228565 84.755602) (end 89.145819 86.070532) (width 0.25) (layer "F.Cu") (net 9))
-  (segment (start 92.92565 87.975224) (end 95.654006 90.971065) (width 0.25) (layer "F.Cu") (net 9))
-  (segment (start 97.485 92.68) (end 98.47 93.46) (width 0.25) (layer "F.Cu") (net 9))
-  (segment (start 73.525 83.61) (end 72.35 82.62) (width 0.25) (layer "F.Cu") (net 9))
-  (arc (start 92.92565 87.975224) (mid 91.211652 86.673771) (end 89.145819 86.070532) (width 0.25) (layer "F.Cu") (net 9))
-  (arc (start 76.228565 84.755602) (mid 74.790401 84.386656) (end 73.525 83.61) (width 0.25) (layer "F.Cu") (net 9))
-  (arc (start 97.485 92.68) (mid 96.534808 91.862704) (end 95.654006 90.971065) (width 0.25) (layer "F.Cu") (net 9))
+  (segment (start 75.099999 84.45) (end 74.852958 84.402492) (width 0.25) (layer "F.Cu") (net 9))
+  (segment (start 93.099999 88.25) (end 93.06096 88.025522) (width 0.25) (layer "F.Cu") (net 9))
+  (segment (start 83.635507 85.765136) (end 90.262924 86.233742) (width 0.25) (layer "F.Cu") (net 9))
+  (segment (start 77.702039 84.939149) (end 78.997183 85.177033) (width 0.25) (layer "F.Cu") (net 9))
+  (segment (start 73.075 83.41) (end 72.35 82.62) (width 0.25) (layer "F.Cu") (net 9))
+  (segment (start 94.218024 90.120924) (end 98.47 93.46) (width 0.25) (layer "F.Cu") (net 9))
+  (arc (start 73.075 83.41) (mid 73.884113 84.049318) (end 74.852958 84.402492) (width 0.25) (layer "F.Cu") (net 9))
+  (arc (start 90.262924 86.233742) (mid 91.178044 86.38415) (end 92.05 86.7) (width 0.25) (layer "F.Cu") (net 9))
+  (arc (start 75.099999 84.45) (mid 76.400509 84.697287) (end 77.702039 84.939149) (width 0.25) (layer "F.Cu") (net 9))
+  (arc (start 78.997183 85.177033) (mid 81.308178 85.535492) (end 83.635507 85.765136) (width 0.25) (layer "F.Cu") (net 9))
+  (arc (start 92.05 86.7) (mid 92.717451 87.239227) (end 93.06096 88.025522) (width 0.25) (layer "F.Cu") (net 9))
+  (arc (start 93.099999 88.25) (mid 93.485669 89.289047) (end 94.218024 90.120924) (width 0.25) (layer "F.Cu") (net 9))
   (segment (start 105.08 62) (end 99.49 57.1275) (width 0.25) (layer "B.Cu") (net 10))
   (segment (start 80.707926 79.241111) (end 77.43 82.62) (width 0.25) (layer "F.Cu") (net 11))
   (segment (start 101.505615 67.265469) (end 101.53 57.1275) (width 0.25) (layer "F.Cu") (net 11))
-  (segment (start 98.178479 74.777159) (end 84.551172 77.199791) (width 0.25) (layer "F.Cu") (net 11))
-  (segment (start 100.933791 71.864833) (end 100.822612 72.309551) (width 0.25) (layer "F.Cu") (net 11))
+  (segment (start 84.551172 77.199791) (end 98.178479 74.777159) (width 0.25) (layer "F.Cu") (net 11))
+  (segment (start 100.822612 72.309551) (end 100.933791 71.864833) (width 0.25) (layer "F.Cu") (net 11))
   (arc (start 100.822612 72.309551) (mid 99.86533 73.934236) (end 98.178479 74.777159) (width 0.25) (layer "F.Cu") (net 11))
   (arc (start 101.505615 67.265469) (mid 101.359334 69.582511) (end 100.933791 71.864833) (width 0.25) (layer "F.Cu") (net 11))
-  (arc (start 84.551172 77.199791) (mid 82.468858 77.917914) (end 80.707926 79.241111) (width 0.25) (layer "F.Cu") (net 11))
+  (arc (start 80.707926 79.241111) (mid 82.468858 77.917914) (end 84.551172 77.199791) (width 0.25) (layer "F.Cu") (net 11))
   (segment (start 85.49 57.1275) (end 91.1 62) (width 0.25) (layer "B.Cu") (net 12))
   (segment (start 78.178782 65.206924) (end 74.89 67.38) (width 0.25) (layer "F.Cu") (net 13))
@@
   (segment (start 66.92 62) (end 67.27 67.38) (width 0.25) (layer "F.Cu") (net 24))
   (segment (start 62.19 67.38) (end 52.94 62) (width 0.25) (layer "F.Cu") (net 25))
-  (segment (start 81.5 74) (end 94.5 74) (width 0.25) (layer "F.Cu") (net 26))
-  (segment (start 57.11 67.38) (end 62 72.5) (width 0.25) (layer "F.Cu") (net 26))
-  (segment (start 62 72.5) (end 81.5 74) (width 0.25) (layer "F.Cu") (net 26))
-  (segment (start 94.5 74) (end 98.75 72) (width 0.25) (layer "F.Cu") (net 26))
+  (segment (start 92.185073 74) (end 83.84228 74) (width 0.25) (layer "F.Cu") (net 26))
+  (segment (start 60.43518 70.861579) (end 57.11 67.38) (width 0.25) (layer "F.Cu") (net 26))
+  (segment (start 64.258957 72.673765) (end 79.164618 73.820355) (width 0.25) (layer "F.Cu") (net 26))
+  (segment (start 96.594588 73.014311) (end 98.75 72) (width 0.25) (layer "F.Cu") (net 26))
+  (arc (start 60.43518 70.861579) (mid 62.179471 72.121308) (end 64.258957 72.673765) (width 0.25) (layer "F.Cu") (net 26))
+  (arc (start 79.164618 73.820355) (mid 81.501725 73.955072) (end 83.84228 74) (width 0.25) (layer "F.Cu") (net 26))
+  (arc (start 96.594588 73.014311) (mid 94.444243 73.750573) (end 92.185073 74) (width 0.25) (layer "F.Cu") (net 26))
   (segment (start 98.75 71.75) (end 98.75 78.25) (width 0.25) (layer "B.Cu") (net 26))
   (segment (start 79.97 82.62) (end 90 78.8) (width 0.25) (layer "F.Cu") (net 27))
