File: pcb/button_v1/kamaji_button_v1.kicad_sch (KiCad schematic)
At the start: 3 parts, among them J1 RJ10, SW2 SW_Push_LED

Commit message: Fix CI
Parts:
- removed D1: LED, LED_THT:LED_D5.0mm, symbol Device:LED
Changed lines of the file:
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@@
 (kicad_sch (version 20211123) (generator eeschema)
   (paper "A4")
-  (junction (at 124.46 90.17) (diameter 0) (color 0 0 0 0)
-  )
   (junction (at 97.79 90.17) (diameter 0) (color 0 0 0 0)
   )
@@
   )
   (wire (pts (xy 97.79 87.63) (xy 102.87 87.63))
-    (stroke (width 0) (type default) (color 0 0 0 0))
-  )
-  (wire (pts (xy 124.46 90.17) (xy 124.46 91.44))
     (stroke (width 0) (type default) (color 0 0 0 0))
   )
@@
   (wire (pts (xy 124.46 83.82) (xy 124.46 90.17))
     (stroke (width 0) (type default) (color 0 0 0 0))
-  )
-  (symbol (lib_id "Device:LED") (at 124.46 95.25 90) (unit 1)
-    (in_bom yes) (on_board yes) (fields_autoplaced)
-    (property "Reference" "D1" (id 0) (at 128.27 95.5674 90)
-      (effects (font (size 1.27 1.27)) (justify right))
-    )
-    (property "Value" "LED" (id 1) (at 128.27 98.1074 90)
-      (effects (font (size 1.27 1.27)) (justify right))
-    )
-    (property "Footprint" "LED_THT:LED_D5.0mm" (id 2) (at 124.46 95.25 0)
-      (effects (font (size 1.27 1.27)) hide)
-    )
-    (property "Datasheet" "~" (id 3) (at 124.46 95.25 0)
-      (effects (font (size 1.27 1.27)) hide)
-    )
-    (pin "1")
-    (pin "2")
-  )
-  (symbol (lib_id "power:GND") (at 124.46 99.06 0) (unit 1)
-    (in_bom yes) (on_board yes) (fields_autoplaced)
-    (property "Reference" "#PWR0104" (id 0) (at 124.46 105.41 0)
-      (effects (font (size 1.27 1.27)) hide)
-    )
-    (property "Value" "GND" (id 1) (at 124.46 104.14 0))
-    (property "Footprint" "" (id 2) (at 124.46 99.06 0)
-      (effects (font (size 1.27 1.27)) hide)
-    )
-    (property "Datasheet" "" (id 3) (at 124.46 99.06 0)
-      (effects (font (size 1.27 1.27)) hide)
-    )
-    (pin "1")
   )
   (symbol (lib_id "power:GND") (at 121.92 83.82 0) (unit 1)
@@
       (reference "#PWR0103") (unit 1) (value "GND") (footprint "")
     )
-    (path "/803f08ac-ffe6-4a8f-a2a2-759bf9dbbb0d"
-      (reference "#PWR0104") (unit 1) (value "GND") (footprint "")
-    )
-    (path "/74af65a9-fc99-45d8-9a9b-08f4a78463fd"
-      (reference "D1") (unit 1) (value "LED") (footprint "LED_THT:LED_D5.0mm")
-    )
     (path "/afdf104e-d29b-4a8d-9f3b-2d2ea2d5b7d6"

Commit message: button pcb: replace the switch footprint
Parts:
- SW2: footprint mx_alps_hybrid:MX-1U -> kamaji:SW_Cherry_MX_1.00u_PCB
Changed lines of the file:
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@@
     (property "Reference" "SW2" (id 0) (at 107.315 80.01 0))
     (property "Value" "SW_Push_LED" (id 1) (at 107.315 82.55 0))
-    (property "Footprint" "mx_alps_hybrid:MX-1U" (id 2) (at 107.95 82.55 0)
+    (property "Footprint" "kamaji:SW_Cherry_MX_1.00u_PCB" (id 2) (at 107.95 82.55 0)
       (effects (font (size 1.27 1.27)) hide)
     )
@@
     )
     (path "/a40da50e-6d7d-4ff7-a5d3-a5cb3c9931e9"
-      (reference "SW2") (unit 1) (value "SW_Push_LED") (footprint "mx_alps_hybrid:MX-1U")
+      (reference "SW2") (unit 1) (value "SW_Push_LED") (footprint "kamaji:SW_Cherry_MX_1.00u_PCB")
     )
   )
