File: pcb/button_v1/kamaji_button_v1.kicad_pcb (KiCad board)
At the start: 2 copper layers, 30 x 35 mm, 4 parts, among them J1 RJ10, SW2 SW_Push_LED

Commit message: Fix CI
Parts:
- removed D1: LED, LED_THT:LED_D5.0mm
- added REF**: MountingHole_3.2mm_M3, MountingHole:MountingHole_3.2mm_M3, F.Cu at (76.5, 83.5)
- added REF**: MountingHole_3.2mm_M3, MountingHole:MountingHole_3.2mm_M3, F.Cu at (53.5, 83.5)
- added REF**: MountingHole_3.2mm_M3, MountingHole:MountingHole_3.2mm_M3, F.Cu at (53.5, 53.5)
- added REF**: MountingHole_3.2mm_M3, MountingHole:MountingHole_3.2mm_M3, F.Cu at (76.5, 53.5)
- J1: moved to F.Cu
- moved SW2 3.00 mm to (65.0, 71.0)
- moved REF** 2.00 mm to (65.0, 83.5)
- turned J1 to 180 degrees
Routing:
- net Net-(J1-Pad2): track 20.6 -> 0.00 mm
- net Net-(J1-Pad4): track 16.9 -> 0.00 mm
Other:
- board size 30 x 35 mm -> 30 x 37 mm

Commit message: Button PCB: minor changes
Parts:
- removed the REF** at (76.5, 83.5)
- removed the REF** at (53.5, 83.5)
- removed the REF** at (53.5, 53.5)
- removed the REF** at (76.5, 53.5)
Changed lines of the file:
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@@
   (net 3 "Net-(J1-Pad2)")
-  (footprint "MountingHole:MountingHole_3.2mm_M3" (layer "F.Cu")
-    (at 76.5 83.5)
-    (descr "Mounting Hole 3.2mm, no annular, M3")
-    (tags "mounting hole 3.2mm no annular m3")
-    (attr exclude_from_pos_files exclude_from_bom)
-    (fp_text reference "REF**" (at 0 -4.2) (layer "F.SilkS") hide
-      (effects (font (size 1 1) (thickness 0.15)))
-    )
-    (fp_text value "MountingHole_3.2mm_M3" (at 0 4.2) (layer "F.Fab") hide
-      (effects (font (size 1 1) (thickness 0.15)))
-    )
-    (fp_text user "${REFERENCE}" (at 0 0) (layer "F.Fab")
-      (effects (font (size 1 1) (thickness 0.15)))
-    )
-    (fp_circle (center 0 0) (end 3.2 0) (layer "Cmts.User") (width 0.15) (fill none))
-    (fp_circle (center 0 0) (end 3.45 0) (layer "F.CrtYd") (width 0.05) (fill none))
-    (pad "" np_thru_hole circle (at 0 0) (size 3.2 3.2) (drill 3.2) (layers *.Cu *.Mask))
-  )
-  (footprint "MountingHole:MountingHole_3.2mm_M3" (layer "F.Cu")
-    (at 53.5 83.5)
-    (descr "Mounting Hole 3.2mm, no annular, M3")
-    (tags "mounting hole 3.2mm no annular m3")
-    (attr exclude_from_pos_files exclude_from_bom)
-    (fp_text reference "REF**" (at 0 -4.2) (layer "F.SilkS") hide
-      (effects (font (size 1 1) (thickness 0.15)))
-    )
-    (fp_text value "MountingHole_3.2mm_M3" (at 0 4.2) (layer "F.Fab") hide
-      (effects (font (size 1 1) (thickness 0.15)))
-    )
-    (fp_text user "${REFERENCE}" (at 0 0) (layer "F.Fab")
-      (effects (font (size 1 1) (thickness 0.15)))
-    )
-    (fp_circle (center 0 0) (end 3.2 0) (layer "Cmts.User") (width 0.15) (fill none))
-    (fp_circle (center 0 0) (end 3.45 0) (layer "F.CrtYd") (width 0.05) (fill none))
-    (pad "" np_thru_hole circle (at 0 0) (size 3.2 3.2) (drill 3.2) (layers *.Cu *.Mask))
-  )
-  (footprint "MountingHole:MountingHole_3.2mm_M3" (layer "F.Cu")
-    (at 53.5 53.5)
-    (descr "Mounting Hole 3.2mm, no annular, M3")
-    (tags "mounting hole 3.2mm no annular m3")
-    (attr exclude_from_pos_files exclude_from_bom)
-    (fp_text reference "REF**" (at 0 -4.2) (layer "F.SilkS") hide
-      (effects (font (size 1 1) (thickness 0.15)))
-    )
-    (fp_text value "MountingHole_3.2mm_M3" (at 0 4.2) (layer "F.Fab") hide
-      (effects (font (size 1 1) (thickness 0.15)))
-    )
-    (fp_text user "${REFERENCE}" (at 0 0) (layer "F.Fab")
-      (effects (font (size 1 1) (thickness 0.15)))
-    )
-    (fp_circle (center 0 0) (end 3.2 0) (layer "Cmts.User") (width 0.15) (fill none))
-    (fp_circle (center 0 0) (end 3.45 0) (layer "F.CrtYd") (width 0.05) (fill none))
-    (pad "" np_thru_hole circle (at 0 0) (size 3.2 3.2) (drill 3.2) (layers *.Cu *.Mask))
-  )
-  (footprint "MountingHole:MountingHole_3.2mm_M3" (layer "F.Cu")
-    (at 76.5 53.5)
-    (descr "Mounting Hole 3.2mm, no annular, M3")
-    (tags "mounting hole 3.2mm no annular m3")
-    (attr exclude_from_pos_files exclude_from_bom)
-    (fp_text reference "REF**" (at 0 -4.2) (layer "F.SilkS") hide
-      (effects (font (size 1 1) (thickness 0.15)))
-    )
-    (fp_text value "MountingHole_3.2mm_M3" (at 0 4.2) (layer "F.Fab") hide
-      (effects (font (size 1 1) (thickness 0.15)))
-    )
-    (fp_text user "${REFERENCE}" (at 0 0) (layer "F.Fab")
-      (effects (font (size 1 1) (thickness 0.15)))
-    )
-    (fp_circle (center 0 0) (end 3.2 0) (layer "Cmts.User") (width 0.15) (fill none))
-    (fp_circle (center 0 0) (end 3.45 0) (layer "F.CrtYd") (width 0.05) (fill none))
-    (pad "" np_thru_hole circle (at 0 0) (size 3.2 3.2) (drill 3.2) (layers *.Cu *.Mask))
-  )
   (footprint "MountingHole:MountingHole_3.2mm_M3" (layer "F.Cu")
     (at 65 83.5)
@@
   )
   (dimension (type aligned) (layer "F.Cu")
-    (pts (xy 80 50) (xy 80 86.5))
+    (pts (xy 80 50) (xy 80 87))
     (height -5)
-    (gr_text "36.5000 mm" (at 83.2 68.25 90) (layer "F.Cu")
+    (gr_text "37.0000 mm" (at 83.2 68.5 90) (layer "F.Cu")
       (effects (font (size 1.5 1.5) (thickness 0.3)))
     )

Commit message: Generate gergers
Routing:
- net Net-(J1-Pad4): track 0.00 -> 30.9 mm
- net Net-(J1-Pad2): track 0.00 -> 9.41 mm
Other:
- board text added: "+"
- board text added: "-"
Changed lines of the file:
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@@
       (layerselection 0x00010fc_ffffffff)
       (disableapertmacros false)
-      (usegerberextensions false)
+      (usegerberextensions true)
       (usegerberattributes true)
       (usegerberadvancedattributes true)
@@
       (viasonmask false)
       (mode 1)
-      (useauxorigin false)
+      (useauxorigin true)
       (hpglpennumber 1)
       (hpglpenspeed 20)
@@
       (plotinvisibletext false)
       (sketchpadsonfab false)
-      (subtractmaskfromsilk false)
+      (subtractmaskfromsilk true)
       (outputformat 1)
       (mirror false)
-      (drillshape 1)
+      (drillshape 0)
       (scaleselection 1)
-      (outputdirectory "")
+      (outputdirectory "gerbers/")
     )
   )
@@
     (descr "Mounting Hole 3.2mm, no annular, M3")
     (tags "mounting hole 3.2mm no annular m3")
+    (clearance 1)
     (attr exclude_from_pos_files exclude_from_bom)
     (fp_text reference "REF**" (at 0 -4.2) (layer "F.SilkS") hide
@@
       (effects (font (size 1 1) (thickness 0.15)))
     )
-    (fp_text value "RJ10" (at 0 -5) (layer "F.SilkS")
+    (fp_text value "RJ10" (at 0 -5.5) (layer "F.SilkS")
       (effects (font (size 1 1) (thickness 0.15)))
     )
@@
     (effects (font (size 1 1) (thickness 0.2)))
   )
-  (dimension (type aligned) (layer "F.Cu")
+  (gr_text "-" (at 66.25 68) (layer "F.SilkS")
+    (effects (font (size 1 1) (thickness 0.2)))
+  )
+  (gr_text "+" (at 63.75 68) (layer "F.SilkS")
+    (effects (font (size 1 1) (thickness 0.2)))
+  )
+  (dimension (type aligned) (layer "Dwgs.User")
     (pts (xy 80 50) (xy 80 87))
     (height -5)
-    (gr_text "37.0000 mm" (at 83.2 68.5 90) (layer "F.Cu")
+    (gr_text "37.0000 mm" (at 83.2 68.5 90) (layer "Dwgs.User")
       (effects (font (size 1.5 1.5) (thickness 0.3)))
     )
@@
     (style (thickness 0.2) (arrow_length 1.27) (text_position_mode 0) (extension_height 0.58642) (extension_offset 0.5) keep_text_aligned)
   )
-  (dimension (type aligned) (layer "F.Cu")
+  (dimension (type aligned) (layer "Dwgs.User")
     (pts (xy 50 50) (xy 80 50))
     (height -6.5)
-    (gr_text "30.0000 mm" (at 65 41.7) (layer "F.Cu")
+    (gr_text "30.0000 mm" (at 65 41.7) (layer "Dwgs.User")
       (effects (font (size 1.5 1.5) (thickness 0.3)))
     )
@@
     (style (thickness 0.2) (arrow_length 1.27) (text_position_mode 0) (extension_height 0.58642) (extension_offset 0.5) keep_text_aligned)
   )
+  (segment (start 72.75 71.060784) (end 72.75 71.996036) (width 0.35) (layer "F.Cu") (net 2))
+  (segment (start 63.295 76.915) (end 62.46 76.08) (width 0.35) (layer "F.Cu") (net 2))
+  (segment (start 66.996036 77.75) (end 65.310868 77.75) (width 0.35) (layer "F.Cu") (net 2))
+  (segment (start 71.7011 66.690986) (end 66.53 56.54) (width 0.35) (layer "F.Cu") (net 2))
+  (segment (start 71.156206 75.843792) (end 70.843792 76.156207) (width 0.35) (layer "F.Cu") (net 2))
+  (arc (start 70.843792 76.156207) (mid 69.078426 77.335786) (end 66.996036 77.75) (width 0.35) (layer "F.Cu") (net 2))
+  (arc (start 63.295 76.915) (mid 64.219888 77.53299) (end 65.310868 77.75) (width 0.35) (layer "F.Cu") (net 2))
+  (arc (start 71.7011 66.690986) (mid 72.484102 68.813823) (end 72.75 71.060784) (width 0.35) (layer "F.Cu") (net 2))
+  (arc (start 72.75 71.996036) (mid 72.335786 74.078426) (end 71.156206 75.843792) (width 0.35) (layer "F.Cu") (net 2))
+  (segment (start 64.49 56.54) (end 63.73 65.92) (width 0.35) (layer "F.Cu") (net 3))
   (zone (net 1) (net_name "GND") (layers F&B.Cu) (hatch edge 0.508)
     (connect_pads (clearance 0.508))

Commit message: Tweak the button PCB
Parts:
- moved J1 0.19 mm to (65.0, 46.2)
Routing:
- net Net-(J1-Pad4): track 30.9 -> 28.9 mm
Changed lines of the file:
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@@
   )
   (footprint "kamaji:RJ10" (layer "F.Cu")
-    (at 65 46 180)
+    (at 65 46.1875 180)
     (property "Sheetfile" "File: kamaji_button_v1.kicad_sch")
     (property "Sheetname" "")
@@
     (style (thickness 0.2) (arrow_length 1.27) (text_position_mode 0) (extension_height 0.58642) (extension_offset 0.5) keep_text_aligned)
   )
-  (segment (start 72.75 71.060784) (end 72.75 71.996036) (width 0.35) (layer "F.Cu") (net 2))
-  (segment (start 63.295 76.915) (end 62.46 76.08) (width 0.35) (layer "F.Cu") (net 2))
-  (segment (start 66.996036 77.75) (end 65.310868 77.75) (width 0.35) (layer "F.Cu") (net 2))
-  (segment (start 71.7011 66.690986) (end 66.53 56.54) (width 0.35) (layer "F.Cu") (net 2))
-  (segment (start 71.156206 75.843792) (end 70.843792 76.156207) (width 0.35) (layer "F.Cu") (net 2))
-  (arc (start 70.843792 76.156207) (mid 69.078426 77.335786) (end 66.996036 77.75) (width 0.35) (layer "F.Cu") (net 2))
-  (arc (start 63.295 76.915) (mid 64.219888 77.53299) (end 65.310868 77.75) (width 0.35) (layer "F.Cu") (net 2))
-  (arc (start 71.7011 66.690986) (mid 72.484102 68.813823) (end 72.75 71.060784) (width 0.35) (layer "F.Cu") (net 2))
-  (arc (start 72.75 71.996036) (mid 72.335786 74.078426) (end 71.156206 75.843792) (width 0.35) (layer "F.Cu") (net 2))
-  (segment (start 64.49 56.54) (end 63.73 65.92) (width 0.35) (layer "F.Cu") (net 3))
+  (segment (start 71.649205 73.91389) (end 71.6 74) (width 0.35) (layer "F.Cu") (net 2))
+  (segment (start 65.474152 76.968826) (end 62.46 76.08) (width 0.35) (layer "F.Cu") (net 2))
+  (segment (start 69.099999 76.468363) (end 69.434764 76.257981) (width 0.35) (layer "F.Cu") (net 2))
+  (segment (start 71.408171 68.207254) (end 66.53 56.7275) (width 0.35) (layer "F.Cu") (net 2))
+  (arc (start 65.474152 76.968826) (mid 67.340923 77.108719) (end 69.099999 76.468363) (width 0.35) (layer "F.Cu") (net 2))
+  (arc (start 71.408171 68.207254) (mid 71.901597 69.626935) (end 72.2 71.1) (width 0.35) (layer "F.Cu") (net 2))
+  (arc (start 71.6 74) (mid 70.656544 75.262436) (end 69.434764 76.257981) (width 0.35) (layer "F.Cu") (net 2))
+  (arc (start 72.2 71.1) (mid 72.155878 72.552215) (end 71.649205 73.91389) (width 0.35) (layer "F.Cu") (net 2))
+  (segment (start 64.49 56.7275) (end 63.73 65.92) (width 0.35) (layer "F.Cu") (net 3))
   (zone (net 1) (net_name "GND") (layers F&B.Cu) (hatch edge 0.508)
     (connect_pads (clearance 0.508))

Commit message: Button PCB v1.1
Parts:
- added G***: LOGO, LOGO, F.Cu at (56.0, 83.5)
- added G***: LOGO, LOGO, F.Cu at (54.8, 57.5)
- added G***: LOGO, LOGO, F.Cu at (75.5, 55.5)
- added G***: LOGO, LOGO, B.Cu at (75.5, 68.5)
Routing:
- net Net-(J1-Pad4): track 28.9 -> 29.8 mm
Other:
- outline, holes or cut-outs redrawn
- board text added: "v1.1 12/2022"
- board text removed: "Kamaji Button v1 github.com/iley/kamaji"
