File: pcb/classic_v1/kamaji_classic_v1.kicad_pcb (KiCad board)
At the start: 2 copper layers, 100 x 100 mm, 31 parts, among them J1 USB_A, J2 USB_B, J4 ISP, J5 P1, J6 P2, J7 P3, J8 P4, J9 P5, Q1 BS170, SW1 SW_Push, SW2 SW_Push, SW3 SW_Push, U1 ATmega328P-P

Commit message: Classic: PCB revision 1.1
Parts:
- moved J2 3.50 mm to (64.8, 108.2)
Routing:
- net VCC: track 286.6 -> 284.9 mm
Changed lines of the file:
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@@
   )
   (footprint "Connector_USB:USB_B_Lumberg_2411_02_Horizontal" (layer "F.Cu")
-    (at 64.7875 111.75 180)
+    (at 64.7875 108.25 180)
     (descr "USB 2.0 receptacle type B, horizontal version, through-hole, https://downloads.lumberg.com/datenblaetter/en/2411_02.pdf")
     (tags "USB B receptacle horizontal through-hole")
@@
   (via (at 98 69.75) (size 0.8) (drill 0.4) (layers "F.Cu" "B.Cu") (free) (net 2))
   (via (at 87 127.75) (size 0.8) (drill 0.4) (layers "F.Cu" "B.Cu") (free) (net 2))
+  (segment (start 66.75 142.75) (end 86.75 142.75) (width 0.5) (layer "F.Cu") (net 3))
   (segment (start 71 61.5) (end 71 65.95878) (width 0.5) (layer "F.Cu") (net 3))
   (segment (start 145.5 108.75) (end 145.5 86.08) (width 0.5) (layer "F.Cu") (net 3))
-  (segment (start 86.75 142.75) (end 88.5 141) (width 0.5) (layer "F.Cu") (net 3))
   (segment (start 67 71.5) (end 67 60.65) (width 0.5) (layer "F.Cu") (net 3))
-  (segment (start 67 109.5375) (end 67 71.5) (width 0.5) (layer "F.Cu") (net 3))
-  (segment (start 64.7875 140.7875) (end 66.75 142.75) (width 0.5) (layer "F.Cu") (net 3))
   (segment (start 69.65 60.15) (end 71 61.5) (width 0.5) (layer "F.Cu") (net 3))
   (segment (start 141.75 112.5) (end 145.5 108.75) (width 0.5) (layer "F.Cu") (net 3))
@@
   (segment (start 67 60.65) (end 67.5 60.15) (width 0.5) (layer "F.Cu") (net 3))
   (segment (start 137.2725 112.5) (end 141.75 112.5) (width 0.5) (layer "F.Cu") (net 3))
-  (segment (start 66.75 142.75) (end 86.75 142.75) (width 0.5) (layer "F.Cu") (net 3))
   (segment (start 58.04 71.46) (end 66.96 71.46) (width 0.5) (layer "F.Cu") (net 3))
+  (segment (start 88.5 141) (end 88.5 139) (width 0.5) (layer "F.Cu") (net 3))
+  (segment (start 86.75 142.75) (end 88.5 141) (width 0.5) (layer "F.Cu") (net 3))
+  (segment (start 64.7875 108.25) (end 64.7875 140.7875) (width 0.5) (layer "F.Cu") (net 3))
   (segment (start 99.2 116.33) (end 99.15 116.38) (width 0.5) (layer "F.Cu") (net 3))
   (segment (start 66.96 71.46) (end 67 71.5) (width 0.5) (layer "F.Cu") (net 3))
-  (segment (start 88.5 141) (end 88.5 139) (width 0.5) (layer "F.Cu") (net 3))
+  (segment (start 67 71.5) (end 67 106.0375) (width 0.5) (layer "F.Cu") (net 3))
+  (segment (start 67 106.0375) (end 64.7875 108.25) (width 0.5) (layer "F.Cu") (net 3))
   (segment (start 101.9 105.72) (end 101.74 105.88) (width 0.5) (layer "F.Cu") (net 3))
   (segment (start 67.5 60.15) (end 69.65 60.15) (width 0.5) (layer "F.Cu") (net 3))
   (segment (start 101.9 102.88) (end 101.9 105.72) (width 0.5) (layer "F.Cu") (net 3))
-  (segment (start 64.7875 111.75) (end 64.7875 140.7875) (width 0.5) (layer "F.Cu") (net 3))
+  (segment (start 64.7875 140.7875) (end 66.75 142.75) (width 0.5) (layer "F.Cu") (net 3))
   (segment (start 99.2 113.5) (end 99.2 116.33) (width 0.5) (layer "F.Cu") (net 3))
-  (segment (start 64.7875 111.75) (end 67 109.5375) (width 0.5) (layer "F.Cu") (net 3))
+  (segment (start 73.75 108.25) (end 80.75 101.25) (width 0.5) (layer "B.Cu") (net 3))
+  (segment (start 64.7875 108.25) (end 73.75 108.25) (width 0.5) (layer "B.Cu") (net 3))
   (segment (start 99.52 118) (end 131.7725 118) (width 0.5) (layer "B.Cu") (net 3))
   (segment (start 83.428961 118.071039) (end 83.5 118) (width 0.5) (layer "B.Cu") (net 3))
-  (segment (start 76.5 118) (end 83.5 118) (width 0.5) (layer "B.Cu") (net 3))
   (segment (start 99.25 117.73) (end 99.52 118) (width 0.5) (layer "B.Cu") (net 3))
+  (segment (start 83.5 118) (end 80.5 118) (width 0.5) (layer "B.Cu") (net 3))
   (segment (start 83.5 118) (end 99.52 118) (width 0.5) (layer "B.Cu") (net 3))
   (segment (start 80.75 101.25) (end 100.27 101.25) (width 0.5) (layer "B.Cu") (net 3))
   (segment (start 131.7725 118) (end 137.2725 112.5) (width 0.5) (layer "B.Cu") (net 3))
-  (segment (start 70.25 111.75) (end 76.5 118) (width 0.5) (layer "B.Cu") (net 3))
   (segment (start 99.15 116.38) (end 99.15 117.63) (width 0.5) (layer "B.Cu") (net 3))
   (segment (start 83.428961 121.260012) (end 83.428961 118.071039) (width 0.5) (layer "B.Cu") (net 3))
-  (segment (start 64.7875 111.75) (end 70.25 111.75) (width 0.5) (layer "B.Cu") (net 3))
-  (segment (start 70.25 111.75) (end 80.75 101.25) (width 0.5) (layer "B.Cu") (net 3))
+  (segment (start 73.75 111.25) (end 73.75 108.25) (width 0.5) (layer "B.Cu") (net 3))
+  (segment (start 80.5 118) (end 73.75 111.25) (width 0.5) (layer "B.Cu") (net 3))
   (segment (start 100.27 101.25) (end 101.9 102.88) (width 0.5) (layer "B.Cu") (net 3))
   (segment (start 99.15 117.63) (end 99.25 117.73) (width 0.5) (layer "B.Cu") (net 3))
