File: pcb/classic_v1/kamaji_classic_v1.kicad_sch (KiCad schematic)
At the start: 25 parts, among them J1 USB_B, J2 USB_A, J3 Buttons, J4 RJ10, J5 RJ10, J6 RJ10, J7 RJ10, J8 RJ10, J9 ISP, Q1 NMOS, U1 ATmega328P-P

Commit message: Classic: Assign footprints and start PCB layout
Parts:
- removed J3: Buttons, symbol Connector_Generic:Conn_01x04
- added SW1, SW2, SW3: SW_Push, Button_Switch_THT:SW_PUSH-12mm, symbol Switch:SW_Push
- BZ1: footprint (none) -> Buzzer_Beeper:Buzzer_12x9.5RM7.6
- C1: renamed from C2; footprint (none) -> Capacitor_THT:C_Disc_D3.8mm_W2.6mm_P2.50mm
- C2: renamed from C3; footprint (none) -> Capacitor_THT:C_Disc_D3.8mm_W2.6mm_P2.50mm
- C3: renamed from C4; footprint (none) -> Capacitor_THT:C_Disc_D3.8mm_W2.6mm_P2.50mm
- J1: renamed from J2; footprint (none) -> Connector_USB:USB_A_CONNFLY_DS1095-WNR0
- J2: renamed from J1; footprint (none) -> Connector_USB:USB_B_Lumberg_2411_02_Horizontal
- J4: renamed from J9; footprint (none) -> Connector_IDC:IDC-Header_2x05_P2.54mm_Horizontal
- J5: renamed from J4; footprint (none) -> kamaji:RJ10
- J6: renamed from J5; footprint (none) -> kamaji:RJ10
- J7: renamed from J6; footprint (none) -> kamaji:RJ10
- J8: renamed from J7; footprint (none) -> kamaji:RJ10
- J9: renamed from J8; footprint (none) -> kamaji:RJ10
- Q1: value NMOS -> BS170; footprint (none) -> Package_TO_SOT_THT:TO-92_Inline
- R1: renamed from R7; value 220 -> 1K; footprint (none) -> Resistor_THT:R_Axial_DIN0207_L6.3mm_D2.5mm_P10.16mm_Horizontal
- R2: renamed from R8; footprint (none) -> Resistor_THT:R_Axial_DIN0207_L6.3mm_D2.5mm_P10.16mm_Horizontal
- R3: renamed from R1; footprint (none) -> Resistor_THT:R_Axial_DIN0207_L6.3mm_D2.5mm_P10.16mm_Horizontal
- R4: renamed from R2; footprint (none) -> Resistor_THT:R_Axial_DIN0207_L6.3mm_D2.5mm_P10.16mm_Horizontal
- R5: renamed from R3; footprint (none) -> Resistor_THT:R_Axial_DIN0207_L6.3mm_D2.5mm_P10.16mm_Horizontal
- R6: renamed from R4; footprint (none) -> Resistor_THT:R_Axial_DIN0207_L6.3mm_D2.5mm_P10.16mm_Horizontal
- R7: renamed from R5; footprint (none) -> Resistor_THT:R_Axial_DIN0207_L6.3mm_D2.5mm_P10.16mm_Horizontal
- R8: renamed from R6; footprint (none) -> Resistor_THT:R_Axial_DIN0207_L6.3mm_D2.5mm_P10.16mm_Horizontal
- RV1: footprint (none) -> Potentiometer_THT:Potentiometer_Vishay_T73YP_Vertical
Connections:
- net CBTN1: now also SW1.1
- net CBTN2: now also SW2.1, SW3.1
- net GND: now also SW1.2, SW2.2, SW3.2
- no-connect marks 9 -> 10
Other:
- note added: "Control buttons"
- note removed: "Control buttons connector"

Commit message: Classic: Finish first pass of routing
Parts:
- J5: value RJ10 -> P1
- J6: value RJ10 -> P2
- J7: value RJ10 -> P3
- J8: value RJ10 -> P4
- J9: value RJ10 -> P5
Connections:
- net CBTN2: no longer SW3.1
- net CBTN3: now also SW3.1
Changed lines of the file:
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@@
     (effects (font (size 1.27 1.27)) (justify left bottom))
   )
-  (label "CBTN2" (at 200.66 116.84 180) (fields_autoplaced)
+  (label "CBTN3" (at 200.66 116.84 180) (fields_autoplaced)
     (effects (font (size 1.27 1.27)) (justify right bottom))
   )
@@
       (effects (font (size 1.27 1.27)) (justify left))
     )
-    (property "Value" "RJ10" (at 39.37 158.115 90)
+    (property "Value" "P1" (at 39.37 158.115 90)
       (effects (font (size 1.27 1.27)) (justify left))
     )
@@
       (effects (font (size 1.27 1.27)) (justify left))
     )
-    (property "Value" "RJ10" (at 63.5 158.115 90)
+    (property "Value" "P2" (at 63.5 158.115 90)
       (effects (font (size 1.27 1.27)) (justify left))
     )
@@
       (effects (font (size 1.27 1.27)) (justify left))
     )
-    (property "Value" "RJ10" (at 135.89 158.115 90)
+    (property "Value" "P5" (at 135.89 158.115 90)
       (effects (font (size 1.27 1.27)) (justify left))
     )
@@
       (effects (font (size 1.27 1.27)) (justify left))
     )
-    (property "Value" "RJ10" (at 87.63 158.115 90)
+    (property "Value" "P3" (at 87.63 158.115 90)
       (effects (font (size 1.27 1.27)) (justify left))
     )
@@
       (effects (font (size 1.27 1.27)) (justify left))
     )
-    (property "Value" "RJ10" (at 111.76 158.115 90)
-      (effects (font (size 1.27 1.27)) (justify left))
-    )
+    (property "Value" "P4" (at 111.76 158.115 90)
+      (effects (font (size 1.27 1.27)) (justify left))
+    )

Commit message: Minor tweaks to the classic PCB
Parts:
- Q1: footprint Package_TO_SOT_THT:TO-92_Inline -> Package_TO_SOT_THT:TO-92_HandSolder
Changed lines of the file:
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@@
   (title_block
     (title "Kamaji Classic")
-    (rev "1.0")
+    (rev "1.1")
   )
   (junction (at 130.81 121.92) (diameter 0) (color 0 0 0 0)
@@
       (effects (font (size 1.27 1.27)) (justify left))
     )
-    (property "Footprint" "Package_TO_SOT_THT:TO-92_Inline" (at 255.27 62.23 0)
-      (effects (font (size 1.27 1.27)) hide)
-    )
+    (property "Footprint" "Package_TO_SOT_THT:TO-92_HandSolder" (at 255.27 62.23 0)
+      (effects (font (size 1.27 1.27)) hide)
+    )

Commit message: Update Classic V1 KiCAD files
Parts:
- J1: footprint Connector_USB:USB_A_CONNFLY_DS1095-WNR0 -> Connector_USB:USB_A_Connfly_DS1095
